Commit message: Fixed indentations and formatting issues, updated elite urdf, updated dependencies

File: mp_components/urdf/arm/elite_arm.urdf.xacro (robot description, xacro)
@@ -5,29 +5,51 @@
 -->
 <robot xmlns:xacro="http://www.ros.org/wiki/xacro" name="elite">
-  <!-- create arm from macro-->
-  <xacro:include filename="$(find ur_description)/urdf/ur_macro.xacro"/>
+  <!-- Set use_gz = true for simulation -->
+  <xacro:arg name="use_gz" default="false"/>
+  <!-- arm parameters -->
   <xacro:arg name="arm_type" default="ec66"/>
-  <xacro:arg name="use_gazebo" default="true"/>
-  <!--Elite arm parameters-->
+  <!-- Include macros -->
+  <xacro:include filename="$(find elite_description)/urdf/xacros/elite_macro.xacro" />
+  <!--Elite arm parameters -->
   <xacro:arg name="tf_prefix" default="$(arg arm_type)"/>
   <xacro:arg name="joint_limit_params_file" default="$(find elite_description)/config/$(arg arm_type)/joint_limits.yaml"/>
   <xacro:arg name="joint_origin_params_file" default="$(find elite_description)/config/$(arg arm_type)/joint_origins.yaml"/>
   <xacro:arg name="link_inertials_params_file" default="$(find elite_description)/config/$(arg arm_type)/link_inertials.yaml"/>
+  <!-- initial positions file for Elite arm-->
   <xacro:arg name="initial_joint_positions_file" default="$(find elite_description)/config/$(arg arm_type)/initial_positions.yaml"/>
-  <!-- create arm -->
-  <xacro:include filename="$(find elite_description)/urdf/macro/elite_macro.xacro" />
+  <!-- Load parameters from YAML file -->
+  <xacro:property
+    name="elite_initial_positions"
+    value="${xacro.load_yaml('$(arg initial_joint_positions_file)')}"
+    />
   <xacro:elite_robot
     name="$(arg arm_type)"
     tf_prefix="$(arg tf_prefix)"
-    arm_parent="cabinet_link"
+    parent="$(arg arm_parent)"
     joint_limits_parameters_file="$(arg joint_limit_params_file)"
-    joint_origins_parameters_file="$(arg joint_origin_params_file)"
-    link_inertials_parameters_file="$(arg link_inertials_params_file)"
+    kinematics_parameters_file="$(arg kinematics_params_file)"
+    physical_parameters_file="$(arg physical_params_file)"
     >
     <origin xyz="0.133 0.0 0.416" rpy="0.0 0.0 -1.5708" />
   </xacro:elite_robot>
-  <!-- If both Elite Arm and Simulation is used -->
-  <xacro:if value="$(arg use_gazebo)">
-    <xacro:include filename="$(find elite_description)/urdf/elite_gazebo_ros2_control.urdf.xacro" />
+  <!-- If gz simulation is used -->
+  <xacro:if value="$(arg use_gz)">
+    <xacro:include filename="$(find elite_description)/urdf/macro/elite_ros2_control_macro.xacro" />
+    <xacro:arg name="simulation_controllers" default="$(find rox_bringup)/configs/elite/$(arg arm_type)/elite_controllers.yaml"/>
+    <gazebo reference="$(arg arm_parent)">
+    </gazebo>
+    <gazebo>
+      <plugin name="gz_ros2_control::GazeboSimROS2ControlPlugin" filename="libgz_ros2_control-system">
+        <parameters>$(arg simulation_controllers)</parameters>
+      </plugin>
+    </gazebo>
+    <!-- Use the Elite_ros2_control macro -->
+    <xacro:elite_ros2_control
+      name="GazeboSimSystem"
+      tf_prefix="$(arg tf_prefix)"
+      plugin="gz_ros2_control/GazeboSimSystem"
+      parameters="$(arg simulation_controllers)"
+      initial_positions="${elite_initial_positions}"
+      />
   </xacro:if>
 </robot>

File: mp_components/urdf/arm/mpo_cabinet_macro.xacro (robot description, xacro)
@@ -8,5 +8,5 @@
     <joint name="${name}_joint" type="fixed">
       <xacro:insert_block name="origin"/>
-      <joint_properties damping="1" friction="1"/>
+      <dynamics damping="1" friction="1"/>
       <parent link="${parent}"/>
       <child link="${name}_link"/>

Commit message: Added meshes for ur dc cabinet, changed the related files to support this update

File: mp_components/urdf/arm/elite_arm.urdf.xacro (robot description, xacro)
@@ -9,4 +9,5 @@
   <!-- arm parameters -->
   <xacro:arg name="arm_type" default="ec66"/>
+  <xacro:property name="arm_height" default="0.416" />
   <!-- Include macros -->
   <xacro:include filename="$(find elite_description)/urdf/xacros/elite_macro.xacro" />
@@ -33,5 +34,5 @@
     physical_parameters_file="$(arg physical_params_file)"
     >
-    <origin xyz="0.133 0.0 0.416" rpy="0.0 0.0 -1.5708" />
+    <origin xyz="0.133 0.0 ${arm_height}" rpy="0.0 0.0 -1.5708" />
   </xacro:elite_robot>
   <!-- If gz simulation is used -->

File: mp_components/urdf/arm/mpo_cabinet_macro.xacro (robot description, xacro)
@@ -12,4 +12,10 @@
       <child link="${name}_link"/>
     </joint>
+    <xacro:if value="${ur_dc == True}">
+      <xacro:property name="cabinet_mesh" value="cabinet_dc" />
+    </xacro:if>
+    <xacro:if value="${ur_dc == False}">
+      <xacro:property name="cabinet_mesh" value="cabinet_ac" />
+    </xacro:if>
     <link name="${name}_link">
       <inertial>
@@ -21,5 +27,5 @@
         <origin rpy="0 0 -1.5708" xyz="0 0 0"/>
         <geometry>
-          <mesh filename="package://mp_components/meshes/cabin.dae" scale="0.001 0.001 0.001"/>
+          <mesh filename="package://mp_components/meshes/${cabinet_mesh}.dae" scale="0.001 0.001 0.001"/>
         </geometry>
       </visual>
@@ -27,5 +33,5 @@
         <origin rpy="0 0 -1.5708" xyz="0 0 0"/>
         <geometry>
-          <mesh filename="package://mp_components/meshes/cabin.dae" scale="0.001 0.001 0.001"/>
+          <mesh filename="package://mp_components/meshes/${cabinet_mesh}.dae" scale="0.001 0.001 0.001"/>
         </geometry>
       </collision>

File: mp_components/urdf/arm/ur_arm.urdf.xacro (robot description, xacro)
@@ -14,4 +14,5 @@
   <!-- arm parameters -->
   <xacro:arg name="arm_type" default="ur10"/>
+  <xacro:property name="arm_height" default="0.416" />
   <xacro:arg name="arm_parent" default="world"/>
   <!-- UR arm parameters -->
@@ -49,5 +50,5 @@
     >
     <!-- position of arm in the world -->
-    <origin xyz="0.133 0.0 0.416" rpy="0.0 0.0 -1.5708" />
+    <origin xyz="0.133 0.0 ${arm_height}" rpy="0.0 0.0 -1.5708" />
   </xacro:ur_robot>
   <!-- this condition is to ensure that ros2_control doesn't interfere with gz_ros2_control during simulation  -->
